File: Electronicz/KiCad/Mechatron/Mechatron_01.kicad_pcb (KiCad board)
At the start: 2 copper layers, 45 x 21 mm, 54 parts, among them J1 Conn_01x15_Socket, J10 Servo_1, J11 Servo_2, J12 Servo_3, J13 V_ESP32, J14 GND_ESP32, J15 Motor_1, J16 Motor_2, J17 Motor_3, J18 Motor_4, J19 V_LED_2, J2 US_Sensor1, J20 V_LED_1, J21 V_LED_top, J22 GND_LED_top, J23 GND_LED_2, J24 GND_LED_1, J25 SD-Card-Reader, J26 AUDIOAMP, J27 Speaker, J28 Conn_01x01_Pin, J29 Conn_01x01_Pin, J3 US_sensor_2, J30 SW, J4 US_sensor3, J5 US_sensor4, J6 US_sensor5, J7 US_sensor6, J8 GND_Battery, J9 V_Battery_Switch, Q1 LR_LED_Sensors, Q2 LR_3, Q3 LR_2, Q4 LR_1, Q5 LED_top, Q6 LED_2, Q7 LED_1

Commit message: pcb design
Parts:
- moved J12 99.3 mm to (78.7, 96.5), turned to -90 degrees
- moved J11 94.2 mm to (78.7, 100.4), turned to -90 degrees
- moved R4 90.8 mm to (99.1, 137.2)
- moved J10 89.2 mm to (78.7, 104.2), turned to -90 degrees
- moved J25 58.2 mm to (95.2, 62.2), turned to 90 degrees
- moved J15 28.0 mm to (124.5, 94.0)
- moved J16 27.7 mm to (124.5, 88.9)
- moved J27 27.1 mm to (124.5, 132.1), turned to 90 degrees
- moved J17 25.0 mm to (124.5, 78.7)
- moved J18 24.8 mm to (124.5, 73.6)
- moved J2 22.9 mm to (81.3, 68.5)
- moved J3 22.9 mm to (81.3, 73.1)
- moved J4 22.9 mm to (81.3, 77.7)
- moved J5 22.9 mm to (81.3, 82.3)
- moved J6 22.9 mm to (81.3, 86.9)
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Routing:
- net Net-(J10-Pin_2): track 23.0 -> 51.1 mm
- net Net-(J18-Pin_2): track 0.00 -> 14.5 mm
- net Net-(J17-Pin_2): track 0.00 -> 14.5 mm
- net Net-(J16-Pin_2): track 0.00 -> 14.5 mm
- net Net-(J15-Pin_2): track 0.00 -> 14.5 mm
- net Net-(J2-Pin_2): track 23.0 -> 37.1 mm
- net Net-(J10-Pin_1): track 0.00 -> 12.2 mm
- net Net-(J11-Pin_1): track 0.00 -> 11.7 mm
- net Net-(J12-Pin_1): track 0.00 -> 11.2 mm
- net Net-(J18-Pin_1): track 0.00 -> 10.3 mm
- net Net-(J17-Pin_1): track 0.00 -> 10.2 mm
- net Net-(J15-Pin_1): track 0.00 -> 10.2 mm
- net Net-(J16-Pin_1): track 0.00 -> 10.2 mm
- net Net-(J2-Pin_1): track 0.00 -> 9.84 mm
- net Net-(J7-Pin_1): track 0.00 -> 9.67 mm
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
Commit message: Create PCB
Parts:
- J2: value US_Sensor1 -> Front
- J25: footprint Connector_PinSocket_2.54mm:PinSocket_1x06_P2.54mm_Vertical -> Library:SDcard_reader
- J3: value US_sensor_2 -> Left_Front
- J4: value US_sensor3 -> Left_Back
- J5: value US_sensor4 -> Back
- J6: value US_sensor5 -> Right_Back
- J7: value US_sensor6 -> Right_Front
- moved Q1 130.6 mm to (64.1, 116.2)
- moved Q2 130.2 mm to (64.1, 123.8)
- moved Q3 129.8 mm to (64.1, 131.4)
- moved Q4 129.5 mm to (64.1, 139.1)
- moved J13 104.0 mm to (111.8, 135.9)
- moved J8 101.6 mm to (139.7, 36.8)
- moved J14 98.0 mm to (116.8, 135.9)
- moved J9 97.2 mm to (152.4, 36.8)
- moved Q5 94.7 mm to (124.1, 119.4), turned to -90 degrees
- moved J22 89.7 mm to (123.8, 136.5), turned to 180 degrees
- moved J21 89.4 mm to (123.8, 128.9), turned to 180 degrees
- moved J24 83.9 mm to (134.3, 136.5), turned to 180 degrees
- moved Rtop1 83.2 mm to (128.9, 123.8), turned to 90 degrees
- moved J28 79.9 mm to (139.7, 94.0)
- moved Q7 79.1 mm to (134.9, 119.4), turned to -90 degrees
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Routing:
- net Net-(J10-Pin_2): track 51.1 -> 364.7 mm, vias 0 -> 2
- net Net-(Q1-C): track 0.00 -> 226.0 mm
- net Net-(J2-Pin_4): track 23.0 -> 238.1 mm, vias 0 -> 4
- net Net-(J10-Pin_3): track 0.00 -> 65.9 mm, vias 0 -> 2
- net Net-(J11-Pin_3): track 0.00 -> 62.8 mm, vias 0 -> 2
- net Net-(J12-Pin_3): track 0.00 -> 61.3 mm, vias 0 -> 2
- net Net-(J13-Pin_1): track 0.00 -> 57.0 mm, vias 0 -> 2
- net Net-(J25-Pin_5): track 0.00 -> 51.8 mm, vias 0 -> 2
- net Net-(J15-Pin_3): track 0.00 -> 48.9 mm
- net Net-(J1-Pad20): track 0.00 -> 44.9 mm, vias 0 -> 2
- net Net-(J25-Pin_3): track 0.00 -> 43.4 mm
- net Net-(J1-Pad22): track 0.00 -> 41.5 mm
- net Net-(J25-Pin_4): track 0.00 -> 36.1 mm
- net Net-(J1-Pad21): track 0.00 -> 30.0 mm
- net Net-(J15-Pin_4): track 0.00 -> 28.0 mm
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Other:
- board outline removed

Commit message: Finishing PCB
Parts:
- added REF**: MountingHole_3.5mm, MountingHole:MountingHole_3.5mm, F.Cu at (145.0, 140.0)
- added REF**: MountingHole_3.5mm, MountingHole:MountingHole_3.5mm, F.Cu at (25.0, 25.0)
- added REF**: MountingHole_3.5mm, MountingHole:MountingHole_3.5mm, F.Cu at (25.0, 140.0)
- added REF**: MountingHole_3.5mm, MountingHole:MountingHole_3.5mm, F.Cu at (145.0, 25.0)
- moved R2 60.2 mm to (99.9, 90.2), turned to 180 degrees
- moved J23 56.9 mm to (106.9, 94.0)
- moved R1 51.9 mm to (89.8, 98.4), turned to 0 degrees
- moved Q6 51.5 mm to (100.6, 94.0), turned to 180 degrees
- moved J19 47.9 mm to (112.0, 94.0)
- moved J24 44.4 mm to (106.9, 101.6)
- moved C5 38.7 mm to (47.9, 116.2)
- moved Q7 38.4 mm to (100.6, 102.2), turned to 180 degrees
- moved C1 37.1 mm to (47.9, 122.6)
- moved C6 35.7 mm to (47.9, 112.4)
- moved J20 35.2 mm to (112.0, 101.6)
- moved Rtop1 33.7 mm to (99.9, 106.7), turned to 180 degrees
- moved C4 33.5 mm to (48.0, 132.1)
- moved C7 33.3 mm to (47.9, 108.6)
- moved J22 32.1 mm to (106.9, 109.2)
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Connections:
- C1 pad 1: Net-(Q4-B) -> Net-(Q1-C)
- C1 pad 2: Net-(J10-Pin_2) -> Net-(J10-Pin_3)
- C2 pad 1: Net-(Q3-B) -> Net-(Q1-C)
- C2 pad 2: Net-(J10-Pin_2) -> Net-(J10-Pin_3)
- C3 pad 1: Net-(Q2-B) -> Net-(Q1-C)
- C3 pad 2: Net-(J10-Pin_2) -> Net-(J10-Pin_3)
- C4 pad 1: Net-(Q1-B) -> Net-(Q1-C)
- C4 pad 2: Net-(J10-Pin_2) -> Net-(J10-Pin_3)
- C5 pad 1: Net-(J10-Pin_3) -> Net-(J10-Pin_2)
- C5 pad 2: Net-(J10-Pin_2) -> Net-(J10-Pin_3)
- C6 pad 1: Net-(J11-Pin_3) -> Net-(J11-Pin_2)
- C6 pad 2: Net-(J10-Pin_2) -> Net-(J10-Pin_3)
- C7 pad 1: Net-(J12-Pin_3) -> Net-(J12-Pin_2)
- C7 pad 2: Net-(J10-Pin_2) -> Net-(J10-Pin_3)
- C8 pad 1: Net-(J2-Pin_4) -> Net-(J19-Pin_1)
- C8 pad 2: Net-(J10-Pin_2) -> Net-(J10-Pin_3)
- C9 pad 1: Net-(J10-Pin_2) -> Net-(J10-Pin_3)
- J1 pad GND: Net-(J10-Pin_2) -> Net-(J10-Pin_3)
- J11 pad 2: Net-(J10-Pin_2) -> Net-(J11-Pin_2)
- J11 pad 3: Net-(J11-Pin_3) -> Net-(J10-Pin_3)
- J12 pad 2: Net-(J10-Pin_2) -> Net-(J12-Pin_2)
- J12 pad 3: Net-(J12-Pin_3) -> Net-(J10-Pin_3)
- J14 pad 1: Net-(J10-Pin_2) -> Net-(J10-Pin_3)
- J2 pad 3: Net-(J10-Pin_2) -> Net-(J10-Pin_3)
- J2 pad 4: Net-(J2-Pin_4) -> Net-(J19-Pin_1)
- J20 pad 1: Net-(J20-Pin_1) -> Net-(J19-Pin_1)
- J21 pad 1: Net-(J21-Pin_1) -> Net-(J19-Pin_1)
- J22 pad 1: Net-(J10-Pin_2) -> Net-(J22-Pin_1)
- J23 pad 1: Net-(J10-Pin_2) -> Net-(J23-Pin_1)
- J24 pad 1: Net-(J10-Pin_2) -> Net-(J24-Pin_1)
- J25 pad 1: Net-(J10-Pin_2) -> Net-(J10-Pin_3)
- J25 pad 2: Net-(J2-Pin_4) -> Net-(J19-Pin_1)
- J25 pad 6: Net-(J10-Pin_2) -> Net-(J10-Pin_3)
- J26 pad 3: Net-(J10-Pin_2) -> Net-(J10-Pin_3)
- J26 pad 6: Net-(J10-Pin_2) -> Net-(J10-Pin_3)
- J26 pad 8: Net-(J10-Pin_2) -> Net-(J10-Pin_3)
- J3 pad 3: Net-(J10-Pin_2) -> Net-(J10-Pin_3)
- J3 pad 4: Net-(J2-Pin_4) -> Net-(J19-Pin_1)
- J4 pad 3: Net-(J10-Pin_2) -> Net-(J10-Pin_3)
- J4 pad 4: Net-(J2-Pin_4) -> Net-(J19-Pin_1)
- J5 pad 3: Net-(J10-Pin_2) -> Net-(J10-Pin_3)
- J5 pad 4: Net-(J2-Pin_4) -> Net-(J19-Pin_1)
- J6 pad 3: Net-(J10-Pin_2) -> Net-(J10-Pin_3)
- J6 pad 4: Net-(J2-Pin_4) -> Net-(J19-Pin_1)
- J7 pad 3: Net-(J10-Pin_2) -> Net-(J10-Pin_3)
- J7 pad 4: Net-(J2-Pin_4) -> Net-(J19-Pin_1)
- J8 pad 1: Net-(J10-Pin_2) -> Net-(J10-Pin_3)
- Q1 pad 2: Net-(Q1-B) -> Net-(J10-Pin_3)
- Q1 pad 3: Net-(J2-Pin_4) -> Net-(J19-Pin_1)
- Q2 pad 2: Net-(Q2-B) -> Net-(J10-Pin_3)
- Q2 pad 3: Net-(J12-Pin_3) -> Net-(J12-Pin_2)
- Q3 pad 2: Net-(Q3-B) -> Net-(J10-Pin_3)
- Q3 pad 3: Net-(J11-Pin_3) -> Net-(J11-Pin_2)
- Q4 pad 2: Net-(Q4-B) -> Net-(J10-Pin_3)
- Q4 pad 3: Net-(J10-Pin_3) -> Net-(J10-Pin_2)
- Q5 pad 1: Net-(J2-Pin_4) -> Net-(J22-Pin_1)
- Q5 pad 3: Net-(J21-Pin_1) -> Net-(J10-Pin_3)
- Q6 pad 1: Net-(J2-Pin_4) -> Net-(J23-Pin_1)
- Q6 pad 3: Net-(J19-Pin_1) -> Net-(J10-Pin_3)
- Q7 pad 1: Net-(J2-Pin_4) -> Net-(J24-Pin_1)
- Q7 pad 3: Net-(J20-Pin_1) -> Net-(J10-Pin_3)
- U1 pad 2: Net-(J10-Pin_2) -> Net-(J10-Pin_3)
Routing:
- net Net-(J10-Pin_2): track 364.7 -> 68.6 mm, vias 2 -> 4
- net Net-(J10-Pin_3): track 65.9 -> 344.6 mm
- net Net-(J2-Pin_4): track 238.1 -> 0.00 mm, vias 4 -> 0
- net Net-(J19-Pin_1): track 7.25 -> 204.4 mm, vias 0 -> 4
- net Net-(J11-Pin_2): track 0.00 -> 63.3 mm, vias 0 -> 4
- net Net-(J11-Pin_3): track 62.8 -> 0.00 mm, vias 2 -> 0
- net Net-(J12-Pin_3): track 61.3 -> 0.00 mm, vias 2 -> 0
- net Net-(J12-Pin_2): track 0.00 -> 59.4 mm, vias 0 -> 4
- net Net-(J1-Pad22): track 41.5 -> 5.79 mm
- net Net-(J1-Pad21): track 30.0 -> 9.13 mm
- net Net-(Q4-B): track 15.1 -> 0.00 mm
- net Net-(Q3-B): track 14.5 -> 0.00 mm
- net Net-(Q1-B): track 13.8 -> 0.00 mm
- net Net-(Q2-B): track 13.3 -> 0.00 mm
- net Net-(J1-Pad20): track 44.9 -> 37.6 mm
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Other:
- board outline added: 130 x 125 mm
- board text added: "Mechatron_5AHME_23/24_Group2 Templ & Kögelberger"

Commit message: export pcb and schematic pdfs
Parts:
- moved J20 24.3 mm to (128.7, 119.3)
- moved C5 24.3 mm to (64.7, 133.9)
- moved C6 24.3 mm to (64.7, 130.1)
- moved C7 24.3 mm to (64.7, 126.3)
- moved J17 24.3 mm to (111.0, 87.5)
- moved J19 24.3 mm to (128.7, 111.7)
- moved J21 24.3 mm to (128.7, 126.9)
- moved J24 24.3 mm to (123.7, 119.3)
- moved J25 24.3 mm to (111.5, 49.1)
- moved J26 24.3 mm to (75.0, 139.6)
- moved J6 24.3 mm to (67.8, 95.7)
- moved Q5 24.3 mm to (117.3, 128.2)
- moved J8 24.3 mm to (126.2, 45.6)
- moved J9 24.3 mm to (138.9, 45.6)
- moved U1 24.3 mm to (143.6, 54.3)
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