File: Electronicz/KiCad/Mechatron/Mechatron_01.kicad_sch (KiCad schematic)
At the start: 54 parts, among them J1 Conn_01x15_Socket, J10 Servo_1, J11 Servo_2, J12 Servo_3, J13 V_ESP32, J14 GND_ESP32, J15 Motor_1, J16 Motor_2, J17 Motor_3, J18 Motor_4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

Commit message: export pcb and schematic pdfs
Connections:
- net at J1.VIN, J13.1 (Pin_1), J26.4 (Pin_4): now also U1.1 (VIN)
- net at C1.1, C2.1, C3.1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: no longer U1.1 (VIN)
Other:
- moved on the sheet: C1, C10, C2, C3, C4, C5, C6, C7, C8, C9, F1, J1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
